Commit message: bug fix

File: mmwave/sensor_tower_description/urdf/sensor_tower.urdf (robot description, URDF)
Before this commit: robot sensor_tower, 6 links, 5 joints
Joints:
- joint mmwave_right_joint: origin xyz=0.082901 -0.13406 0.14446 rpy=0 0 -1.5708 -> xyz=0.082901 -0.13406 0.14446 rpy=0 0 -0.7854
